Commit message: Update rplidar.xacro

File: hhbot_description/urdf/rplidar.xacro (robot description, xacro)
@@ -24,38 +24,4 @@
             </collision>
         </link>
-        <gazebo reference="${prefix}_link">
-            <material>Gazebo/Black</material>
-        </gazebo>
-        <gazebo reference="${prefix}_link">
-            <sensor type="ray" name="rplidar">
-                <pose>0 0 0 0 0 0</pose>
-                <visualize>false</visualize>
-                <update_rate>5.5</update_rate>
-                <ray>
-                    <scan>
-                      <horizontal>
-                        <samples>360</samples>
-                        <resolution>1</resolution>
-                        <min_angle>-3</min_angle>
-                        <max_angle>3</max_angle>
-                      </horizontal>
-                    </scan>
-                    <range>
-                      <min>0.1</min>
-                      <max>6.0</max>
-                      <resolution>0.01</resolution>
-                    </range>
-                    <noise>
-                      <type>gaussian</type>
-                      <mean>0.0</mean>
-                      <stddev>0.01</stddev>
-                    </noise>
-                </ray>
-                <plugin name="gazebo_rplidar" filename="libgazebo_ros_laser.so">
-                    <topicName>/scan</topicName>
-                    <frameName>laser_link</frameName>
-                </plugin>
-            </sensor>
-        </gazebo>
     </xacro:macro>
 </robot>
