Commit message: Add files via upload

File: hhbot_description/urdf/camera.xacro (robot description, xacro)
@@ -1,6 +1,5 @@
 <?xml version="1.0"?>
-<robot xmlns:xacro="http://www.ros.org/wiki/xacro" name="laser">
-    <xacro:macro name="rplidar" params="prefix:=laser">
-        <!-- Create laser reference frame -->
+<robot xmlns:xacro="http://www.ros.org/wiki/xacro" name="camera">
+    <xacro:macro name="usb_camera" params="prefix:=camera">
         <link name="${prefix}_link">
             <inertial>
@@ -8,17 +7,18 @@
                 <origin xyz="0 0 0" />
                 <inertia ixx="0.01" ixy="0.0" ixz="0.0"
-                         iyy="0.01" iyz="0.0" izz="0.01" />
+                         iyy="0.01" iyz="0.0"
+                         izz="0.01" />
             </inertial>
             <visual>
-                <origin xyz=" 0 0 -0.01 " rpy="0 0 0" />
+                <origin xyz=" 0 0 0 " rpy="0 0 0" />
                 <geometry>
-                    <cylinder length="0.03" radius="0.035"/>
+                    <box size="0.01 0.03 0.03" />
                 </geometry>
-                <material name="black"/>
+                <material name="Black"/>
             </visual>
             <collision>
                 <origin xyz="0.0 0.0 0.0" rpy="0 0 0" />
                 <geometry>
-                    <cylinder length="0.03" radius="0.035"/>
+                    <box size="0.01 0.03 0.03" />
                 </geometry>
             </collision>

File: hhbot_description/urdf/hhbot.urdf (robot description, URDF)
Before this commit: robot hhbot, 6 links, 5 joints
Links:
- link tail: geometry visual box size=0.02 0.1 0.02
Joints:
- joint left_back_wheel_joint: origin xyz=-0.07 -0.1 -0.02 rpy=0 1.57075 0 -> xyz=-0.1 -0.07 -0.02 rpy=1.57075 0 0
- joint left_front_wheel_joint: origin xyz=-0.07 0.1 -0.02 rpy=0 1.57075 0 -> xyz=0.1 -0.07 -0.02 rpy=1.57075 0 0
- joint right_back_wheel_joint: origin xyz=0.07 -0.1 -0.02 rpy=0 1.57075 0 -> xyz=-0.1 0.07 -0.02 rpy=1.57075 0 0
- joint right_front_wheel_joint: origin xyz=0.07 0.1 -0.02 rpy=0 1.57075 0 -> xyz=0.1 0.07 -0.02 rpy=1.57075 0 0
- joint tail_joint: origin xyz=0 -0.09 0.023 rpy=1.0472 0 0 -> xyz= -0.09 0 0.023 rpy=0 -1.0472 0

File: hhbot_description/urdf/hhbot_body.urdf.xacro (robot description, xacro)
@@ -25,9 +25,9 @@
     <xacro:property name="wheel_centre" value="0.005" />
     <!-- tail length, width, height, y and radian -->
-    <xacro:property name="tail_length" value="0.02" />
-    <xacro:property name="tail_width"  value="0.1" />
+    <xacro:property name="tail_width"  value="0.02" />
+    <xacro:property name="tail_length" value="0.1" />
     <xacro:property name="tail_height" value="0.02" />
-    <xacro:property name="tail_y"      value="-0.09" />
-    <xacro:property name="tail_radian" value="1.0472" />
+    <xacro:property name="tail_x"      value="-0.09" />
+    <xacro:property name="tail_radian" value="-1.0472" />
     <!-- Macro for inertia matrix -->
     <xacro:macro name="sphere_inertial_matrix" params="m r">
@@ -88,8 +88,8 @@
             <parent link="base_link" />
             <child link="${lr}_${fb}_wheel_link" />
-            <origin xyz="${sign_lr*base_link_width/2}
-                         ${sign_fb*(base_link_length/2-wheel_radius)}
+            <origin xyz="${sign_fb*(base_link_length/2-wheel_radius)}
+                         ${sign_lr*base_link_width/2}
                          ${wheel_centre-wheel_radius}"
-                    rpy="0 ${H_PI/2} 0" />
+                    rpy="${H_PI/2} 0 0" />
         </joint>
     </xacro:macro>
@@ -107,5 +107,5 @@
             <parent link="base_link"/>
             <child link="tail_link"/>
-            <origin rpy="${tail_radian} 0 0" xyz="0 ${tail_y} ${base_link_height/2-0.002}"/>
+            <origin rpy="0 ${tail_radian} 0" xyz="${tail_x} 0 ${base_link_height/2-0.002}"/>
         </joint>
     </xacro:macro>
@@ -115,5 +115,5 @@
         <link name="base_footprint">
             <visual>
-                <origin xyz="0 0 0" rpy="0 0 ${-H_PI/2} " />
+                <origin xyz="0 0 0" rpy="0 0 0 " />
                 <geometry>
                     <box size="0.001 0.001 0.001" />
@@ -122,5 +122,5 @@
         </link>
         <joint name="base_footprint_joint" type="fixed">
-            <origin xyz="0 0 ${base_link_height/2+wheel_radius-wheel_centre}" rpy="0 0 ${-H_PI/2}" />
+            <origin xyz="0 0 ${base_link_height/2+wheel_radius-wheel_centre}" rpy="0 0 0" />
             <parent link="base_footprint"/>
             <child link="base_link" />
@@ -130,5 +130,5 @@
         <link name="base_link">
             <visual>
-                <origin xyz=" 0 0 0" rpy="0 0 ${H_PI/2}" />
+                <origin xyz=" 0 0 0" rpy="0 0 0" />
                 <geometry>
                     <box size="${base_link_length} ${base_link_width} ${base_link_height}" />
@@ -137,5 +137,5 @@
             </visual>
             <collision>
-                <origin xyz="0 0 0" rpy="0 0 ${H_PI/2}" />
+                <origin xyz="0 0 0" rpy="0 0 0" />
                 <geometry>
                     <box size="${base_link_length} ${base_link_width} ${base_link_height}" />

File: hhbot_description/urdf/hhbot_laser.xacro (robot description, xacro)
@@ -3,6 +3,6 @@
     <xacro:include filename="$(find hhbot_description)/urdf/hhbot_body.urdf.xacro" />
     <xacro:include filename="$(find hhbot_description)/urdf/rplidar.xacro" />
-    <xacro:property name="rplidar_offset_x" value="0" />
-    <xacro:property name="rplidar_offset_y" value="0.05" />
+    <xacro:property name="rplidar_offset_x" value="0.05" />
+    <xacro:property name="rplidar_offset_y" value="0" />
     <!-- Body of hhobot -->
     <hhbot_body/>
